Commit message: simple robot can now be viewed with rviz using urdf and xacro

File: ros2/ros2_ws/install/simple_robot/share/simple_robot/urdf/simple_robot_xacro.urdf.xacro (robot description, xacro)
@@ -1,13 +1,15 @@
 <?xml version="1.0"?>
 <robot name="simple_robot" xmlns:xacro="http://www.ros.org/wiki/xacro">
-  <xacro:property name="wheel_radius" value="0.05" />
+  <xacro:property name="wheel_radius" value="0.1" />
   <xacro:property name="wheel_length" value="0.05" />
+  <xacro:property name="base_size" value="1.0 0.95 0.1" />
+  <xacro:property name="base_origin" value="0 0 0.1" />
   <!-- Base link (rectangle) -->
   <link name="base_link">
     <visual>
       <geometry>
-        <box size="0.6 0.4 0.1"/>
+        <box size="${base_size}"/>
       </geometry>
-      <origin xyz="0 0 0" rpy="0 0 0"/>
+      <origin xyz="${base_origin}" rpy="0 0 0"/>
       <material name="blue">
         <color rgba="0 0 1 1"/>
@@ -16,5 +18,5 @@
     <collision>
       <geometry>
-        <box size="0.6 0.4 0.1"/>
+        <box size="${base_size}"/>
       </geometry>
     </collision>
@@ -77,5 +79,5 @@
     <child link="left_wheel"/>
     <origin xyz="0.0 0.25 0.0" rpy="0 0 0"/>
-    <axis xyz="0 0 1"/>
+    <axis xyz="0 1 0"/>
     <limit effort="1.0" velocity="1.0" lower="-1.5708" upper="1.5708"/>
   </joint>
@@ -85,5 +87,5 @@
     <child link="right_wheel"/>
     <origin xyz="0.0 -0.25 0.0" rpy="0 0 0"/>
-    <axis xyz="0 0 1"/>
+    <axis xyz="0 1 0"/>
     <limit effort="1.0" velocity="1.0" lower="-1.5708" upper="1.5708"/>
   </joint>

Commit message: changed wheel joint to continuous

File: ros2/ros2_ws/install/simple_robot/share/simple_robot/urdf/simple_robot_xacro.urdf.xacro (robot description, xacro)
@@ -75,18 +75,18 @@
   </link>
   <!-- Left wheel joint -->
-  <joint name="left_wheel_joint" type="revolute">
+  <joint name="left_wheel_joint" type="continuous">
     <parent link="base_link"/>
     <child link="left_wheel"/>
     <origin xyz="0.0 0.25 0.0" rpy="0 0 0"/>
     <axis xyz="0 1 0"/>
-    <limit effort="1.0" velocity="1.0" lower="-1.5708" upper="1.5708"/>
+    <!-- <limit effort="1.0" velocity="1.0" lower="-1.5708" upper="1.5708"/> -->
   </joint>
   <!-- Right wheel joint -->
-  <joint name="right_wheel_joint" type="revolute">
+  <joint name="right_wheel_joint" type="continuous">
     <parent link="base_link"/>
     <child link="right_wheel"/>
     <origin xyz="0.0 -0.25 0.0" rpy="0 0 0"/>
     <axis xyz="0 1 0"/>
-    <limit effort="1.0" velocity="1.0" lower="-1.5708" upper="1.5708"/>
+    <!-- <limit effort="1.0" velocity="1.0" lower="-1.5708" upper="1.5708"/> -->
   </joint>
 </robot>
