Commit message: added friction to the wheels

File: ros2/ros2_ws/src/gazebo_robot/urdf/gazebo_robot_xacro.urdf.xacro (robot description, xacro)
@@ -53,4 +53,5 @@
                izz="0.001"/>
     </inertial>
+    <dynamics damping="0.7" friction="0.2"/>
   </link>
    <!-- Right wheel -->
@@ -75,4 +76,5 @@
                izz="0.001"/>
     </inertial>
+    <dynamics damping="0.7" friction="0.2"/>
   </link>
   <!-- Left wheel joint -->
